File: modbusBoard/rs485.brd (EAGLE design)
At the start: 17.1 x 44.1 mm, 13 parts, among them J1 RJ45, U1 MAX485CSA

Commit message: update skematik board
Routing:
- net GND: track 70.7 -> 82.3 mm
Changed lines of the file:
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@@
 <wire x1="14.6822" y1="42.2272" x2="13.7294" y2="43.18" width="0.6096" layer="16"/>
 <wire x1="14.625" y1="28.551625" x2="14.625" y2="26.775" width="0.6096" layer="16"/>
-<wire x1="14.625" y1="26.775" x2="13.335" y2="25.485" width="0.6096" layer="16"/>
+<wire x1="14.625" y1="26.775" x2="13.5975" y2="25.7475" width="0.6096" layer="16"/>
+<wire x1="13.5975" y1="25.7475" x2="13.335" y2="25.485" width="0.6096" layer="16"/>
 <wire x1="13.335" y1="24.195" x2="13.335" y2="25.485" width="0.6096" layer="16"/>
 <wire x1="14.625" y1="28.551625" x2="14.6822" y2="28.608825" width="0.6096" layer="16"/>
@@
 <wire x1="3.265" y1="28.875" x2="3.265" y2="34.19" width="0.6096" layer="16"/>
 <wire x1="3.265" y1="34.19" x2="3.165" y2="34.29" width="0.6096" layer="16"/>
-<wire x1="1.21" y1="43.18" x2="2.62" y2="37.76" width="0" layer="19" extent="16-16"/>
+<wire x1="13.5975" y1="25.7475" x2="11.6422" y2="27.7028" width="0.6096" layer="16"/>
+<wire x1="11.6422" y1="27.7028" x2="9.083825" y2="27.7028" width="0.6096" layer="16"/>
+<wire x1="7.911625" y1="28.875" x2="3.265" y2="28.875" width="0.6096" layer="16"/>
+<wire x1="9.083825" y1="27.7028" x2="7.911625" y2="28.875" width="0.6096" layer="16"/>
 </signal>
 <signal name="N$1">
